File: Electrobot_H755.kicad_pcb (KiCad board)
At the start: 2 copper layers, 88.3 x 136 mm, 223 parts, among them J1 Conn_XT30M, J10 Conn_01x04, J11 Conn_01x04, J12 Conn_01x04, J13 Conn_01x04, J14 Conn_01x04, J15 Conn_01x03, J16 Conn_01x03, J17 Conn_01x04, J18 Conn_01x03, J19 Conn_01x03, J2 Conn_01x04, J20 Conn_01x03, J21 Conn_01x03, J22 Conn_01x04, J23 Conn_01x03, J24 Conn_01x03, J25 Conn_01x03, J26 Conn_01x03, J27 Conn_01x02, J28 Conn_01x02, J29 Conn_01x02, J3 Conn_01x04, J30 Conn_01x02, J31 Conn_01x03, J32 Conn_01x03, J33 Conn_01x06, J34 Conn_01x06, J35 Conn_01x04, J36 Conn_01x02, J37 Conn_01x04, J4 Conn_01x04, J5 Conn_01x04, J6 Conn_01x04, J7 Conn_01x04, J8 Conn_01x04, J9 Conn_01x04, U2 TSR_2-2450, U3 TSR_2-2465, U4 TSR_2-2465

Commit message: Mise à jour sérigraphie manquante
Other:
- board text added: "3.3V"
- board text added: "5V"
- board text added: "B"
- board text added: "P"
- board text added: "Servos"
- board text added: "Vservo1"
- board text added: "Vservo2"
- board text removed: "Servo"
Changed lines of the file:
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@@
 	)
 	(gr_text "+3.3V"
-		(at 140.4112 160.5788 0)
+		(at 140.5128 160.5788 0)
 		(layer "B.SilkS")
 		(effects
@@
 		)
 	)
+	(gr_text "Vservo2"
+		(at 120.9548 48.7172 0)
+		(layer "B.SilkS")
+		(effects
+			(font
+				(size 0.8 0.8)
+				(thickness 0.1)
+				(italic yes)
+			)
+			(justify left bottom mirror)
+		)
+	)
 	(gr_text "+"
 		(at 92.9132 84.4296 90)
@@
 	)
 	(gr_text "+5V"
-		(at 136.398 156.4132 0)
+		(at 136.4996 156.21 0)
 		(layer "B.SilkS")
 		(effects
@@
 		)
 	)
+	(gr_text "Vservo1"
+		(at 120.9548 50.4952 0)
+		(layer "B.SilkS")
+		(effects
+			(font
+				(size 0.8 0.8)
+				(thickness 0.1)
+				(italic yes)
+			)
+			(justify left bottom mirror)
+		)
+	)
 	(gr_text "5"
 		(at 127.5588 47.6504 0)
@@
 		)
 	)
+	(gr_text "B"
+		(at 119.126 88.2904 0)
+		(layer "B.SilkS")
+		(effects
+			(font
+				(size 1 1)
+				(thickness 0.1)
+			)
+			(justify left bottom mirror)
+		)
+	)
 	(gr_text "GND"
 		(at 140.208 155.194 90)
@@
 		)
 	)
+	(gr_text "P"
+		(at 88.9508 127.1524 0)
+		(layer "B.SilkS")
+		(effects
+			(font
+				(size 1 1)
+				(thickness 0.1)
+			)
+			(justify left bottom mirror)
+		)
+	)
 	(gr_text "3"
 		(at 127.5588 54.2544 0)
@@
 		)
 	)
+	(gr_text "A"
+		(at 121.5136 105.5116 0)
+		(layer "B.SilkS")
+		(effects
+			(font
+				(size 1 1)
+				(thickness 0.1)
+			)
+			(justify left bottom mirror)
+		)
+	)
+	(gr_text "P"
+		(at 81.9404 135.4836 0)
+		(layer "B.SilkS")
+		(effects
+			(font
+				(size 1 1)
+				(thickness 0.1)
+			)
+			(justify left bottom mirror)
+		)
+	)
 	(gr_text "+"
 		(at 118.11 142.1384 90)
@@
 	)
 	(gr_text "I2C_SCL"
-		(at 141.986 165.6588 0)
+		(at 142.0368 165.6588 0)
 		(layer "B.SilkS")
 		(effects
@@
 		)
 	)
+	(gr_text "A"
+		(at 121.666 130.302 0)
+		(layer "B.SilkS")
+		(effects
+			(font
+				(size 1 1)
+				(thickness 0.1)
+			)
+			(justify left bottom mirror)
+		)
+	)
+	(gr_text "P"
+		(at 127.254 108.8136 90)
+		(layer "B.SilkS")
+		(effects
+			(font
+				(size 1 1)
+				(thickness 0.1)
+			)
+			(justify left bottom mirror)
+		)
+	)
+	(gr_text "A"
+		(at 121.7168 88.2904 0)
+		(layer "B.SilkS")
+		(effects
+			(font
+				(size 1 1)
+				(thickness 0.1)
+			)
+			(justify left bottom mirror)
+		)
+	)
+	(gr_text "B"
+		(at 118.9228 105.5116 0)
+		(layer "B.SilkS")
+		(effects
+			(font
+				(size 1 1)
+				(thickness 0.1)
+			)
+			(justify left bottom mirror)
+		)
+	)
 	(gr_text "Eana"
 		(at 115.2652 136.9568 90)
@@
 		)
 	)
+	(gr_text "+"
+		(at 114.0968 128.8288 90)
+		(layer "B.SilkS")
+		(effects
+			(font
+				(size 1 1)
+				(thickness 0.1)
+			)
+			(justify left bottom mirror)
+		)
+	)
 	(gr_text "Codeur1"
 		(at 111.2012 97.4852 90)
@@
 	)
 	(gr_text "GND"
-		(at 138.938 168.2496 0)
-		(layer "B.SilkS")
-		(effects
-			(font
-				(size 1 1)
-				(thickness 0.1)
-				(italic yes)
+		(at 139.192 168.2496 0)
+		(layer "B.SilkS")
+		(effects
+			(font
+				(size 1 1)
+				(thickness 0.1)
+				(italic yes)
+			)
+			(justify left bottom mirror)
+		)
+	)
+	(gr_text "A"
+		(at 124.0536 69.6976 0)
+		(layer "B.SilkS")
+		(effects
+			(font
+				(size 1 1)
+				(thickness 0.1)
 			)
 			(justify left bottom mirror)
@@
 	)
 	(gr_text "-"
-		(at 116.6368 104.2924 90)
+		(at 116.6368 104.1908 90)
 		(layer "B.SilkS")
 		(effects
@@
 		)
 	)
+	(gr_text "5V"
+		(at 81.8896 99.8728 90)
+		(layer "B.SilkS")
+		(effects
+			(font
+				(size 0.8 0.8)
+				(thickness 0.1)
+				(italic yes)
+			)
+			(justify left bottom mirror)
+		)
+	)
 	(gr_text "K"
 		(at 122.8852 150.4188 0)
@@
 	)
 	(gr_text "I2C_SDA"
-		(at 142.0368 163.0172 0)
+		(at 142.0876 163.1188 0)
 		(layer "B.SilkS")
 		(effects
@@
 		)
 	)
+	(gr_text "P"
+		(at 89.0524 133.2992 0)
+		(layer "B.SilkS")
+		(effects
+			(font
+				(size 1 1)
+				(thickness 0.1)
+			)
+			(justify left bottom mirror)
+		)
+	)
 	(gr_text "-"
 		(at 81.026 97.79 180)
@@
 		)
 	)
-	(gr_text "Servo"
+	(gr_text "3.3V"
+		(at 82.042 94.1832 90)
+		(layer "B.SilkS")
+		(effects
+			(font
+				(size 0.8 0.8)
+				(thickness 0.1)
+				(italic yes)
+			)
+			(justify left bottom mirror)
+		)
+	)
+	(gr_text "Servos"
 		(at 133.9596 38.6588 0)
 		(layer "B.SilkS")
@@
 		)
 	)
+	(gr_text "B"
+		(at 119.0752 130.302 0)
+		(layer "B.SilkS")
+		(effects
+			(font
+				(size 1 1)
+				(thickness 0.1)
+			)
+			(justify left bottom mirror)
+		)
+	)
+	(gr_text "B"
+		(at 121.4628 69.6976 0)
+		(layer "B.SilkS")
+		(effects
+			(font
+				(size 1 1)
+				(thickness 0.1)
+			)
+			(justify left bottom mirror)
+		)
+	)
 	(gr_text "-"
 		(at 118.872 68.58 90)
@@
 	)
 	(gr_text "USB host"
-		(at 85.598 170.942 -0)
+		(at 85.4456 170.942 -0)
 		(layer "F.SilkS")
 		(effects
@@
 	(via
 		(at 99.314 70.612)
-		(size 0.6)
-		(drill 0.3)
+		(size 1.2)
+		(drill 0.6)
 		(layers "F.Cu" "B.Cu")
 		(net 11)

Commit message: Sérigraphie complétée
Other:
- board text added: "->"
- board text added: "<-"
- board text added: "Codeurs: J7, J8, J9, J10 Moteurs: J2, J3, J4, J5 Servos: J18, J19, J20, J21, J23, J24, J25 Etor: J27, J28, J29, J30 Eana: J15, J16, J17, J26 RS232: J6, J22"
- board text added: "Connecteurs"
- board text added: "LED RGB"
- board text added: "R"
Changed lines of the file:
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@@
 		(tags "connector Molex KK-254 vertical")
 		(property "Reference" "J6"
-			(at 3.81 4.465 90)
+			(at 6.9114 4.3994 90)
 			(layer "B.SilkS")
 			(effects
@@
 	)
 	(gr_line
+		(start 124.8156 48.7172)
+		(end 140.1064 48.7172)
+		(stroke
+			(width 0.1)
+			(type dash)
+		)
+		(layer "B.SilkS")
+	)
+	(gr_line
 		(start 88.4428 75.184)
 		(end 88.4428 94.3864)
@@
 	)
 	(gr_text "-"
-		(at 116.586 87.122 90)
+		(at 116.586 86.9188 90)
 		(layer "B.SilkS")
 		(effects
@@
 		)
 	)
+	(gr_text "Connecteurs"
+		(at 97.3836 143.4592 0)
+		(layer "B.SilkS")
+		(effects
+			(font
+				(size 1 1)
+				(thickness 0.2)
+				(bold yes)
+			)
+			(justify left bottom mirror)
+		)
+	)
 	(gr_text "7"
 		(at 127.5588 40.9956 0)
@@
 		)
 	)
+	(gr_text "LED RGB"
+		(at 101.1936 96.2152 90)
+		(layer "B.SilkS")
+		(effects
+			(font
+				(size 1 1)
+				(thickness 0.1)
+				(italic yes)
+			)
+			(justify left bottom mirror)
+		)
+	)
 	(gr_text "K"
 		(at 116.078 150.368 0)
@@
 		)
 	)
+	(gr_text "<-"
+		(at 91.4908 107.3912 180)
+		(layer "B.SilkS")
+		(effects
+			(font
+				(size 1 1)
+				(thickness 0.1)
+			)
+			(justify left bottom mirror)
+		)
+	)
 	(gr_text "Vservo1"
 		(at 120.9548 50.4952 0)
@@
 		)
 	)
+	(gr_text "Vservo1"
+		(at 141.8336 51.9176 90)
+		(layer "B.SilkS")
+		(effects
+			(font
+				(size 0.8 0.8)
+				(thickness 0.1)
+				(italic yes)
+			)
+			(justify left bottom mirror)
+		)
+	)
 	(gr_text "P"
 		(at 88.9508 127.1524 0)
@@
 	)
 	(gr_text "+"
-		(at 114.1984 87.1728 90)
+		(at 114.1984 86.9696 90)
+		(layer "B.SilkS")
+		(effects
+			(font
+				(size 1 1)
+				(thickness 0.1)
+			)
+			(justify left bottom mirror)
+		)
+	)
+	(gr_text "<-"
+		(at 139.446 104.394 -90)
 		(layer "B.SilkS")
 		(effects
@@
 		)
 	)
+	(gr_text "Vservo2"
+		(at 141.986 42.164 90)
+		(layer "B.SilkS")
+		(effects
+			(font
+				(size 0.8 0.8)
+				(thickness 0.1)
+				(italic yes)
+			)
+			(justify left bottom mirror)
+		)
+	)
 	(gr_text "A"
-		(at 124.0536 69.6976 0)
+		(at 124.0536 78.0288 0)
 		(layer "B.SilkS")
 		(effects
@@
 	)
 	(gr_text "+"
-		(at 113.8936 104.0384 90)
+		(at 113.8936 104.14 90)
 		(layer "B.SilkS")
 		(effects
@@
 	)
 	(gr_text "+"
-		(at 116.5352 68.4784 90)
+		(at 116.5352 76.6572 90)
 		(layer "B.SilkS")
 		(effects
@@
 		)
 	)
+	(gr_text "->"
+		(at 91.5416 109.8296 180)
+		(layer "B.SilkS")
+		(effects
+			(font
+				(size 1 1)
+				(thickness 0.1)
+			)
+			(justify left bottom mirror)
+		)
+	)
 	(gr_text "TX"
 		(at 102.616 108.5088 0)
@@
 		)
 	)
+	(gr_text "->"
+		(at 136.906 104.394 -90)
+		(layer "B.SilkS")
+		(effects
+			(font
+				(size 1 1)
+				(thickness 0.1)
+			)
+			(justify left bottom mirror)
+		)
+	)
 	(gr_text "+"
 		(at 97.8916 102.4636 90)
@@
 		)
 	)
+	(gr_text "Codeurs: J7, J8, J9, J10\nMoteurs: J2, J3, J4, J5\nServos: J18, J19, J20, J21, J23, J24, J25\nEtor: J27, J28, J29, J30\nEana: J15, J16, J17, J26\nRS232: J6, J22\n"
+		(at 97.536 153.3652 0)
+		(layer "B.SilkS")
+		(effects
+			(font
+				(size 1 1)
+				(thickness 0.1)
+			)
+			(justify left bottom mirror)
+		)
+	)
 	(gr_text "P"
 		(at 89.0524 133.2992 0)
@@
 		)
 	)
+	(gr_text "R"
+		(at 82.1944 87.5284 0)
+		(layer "B.SilkS")
+		(effects
+			(font
+				(size 1 1)
+				(thickness 0.1)
+			)
+			(justify left bottom mirror)
+		)
+	)
 	(gr_text "ELECTROBOT_H755 V1\n(2025)"
 		(at 70.0024 58.8264 90)
@@
 	)
 	(gr_text "B"
-		(at 121.4628 69.6976 0)
+		(at 121.4628 78.0288 0)
 		(layer "B.SilkS")
 		(effects
@@
 	)
 	(gr_text "-"
-		(at 118.872 68.58 90)
+		(at 118.872 76.7588 90)
 		(layer "B.SilkS")
 		(effects
@@
 		)
 	)
+	(gr_text "-"
+		(at 83.4136 38.9128 180)
+		(layer "F.SilkS")
+		(effects
+			(font
+				(size 1 1)
+				(thickness 0.1)
+			)
+			(justify left bottom mirror)
+		)
+	)
 	(gr_text "USB\nSTLINK"
 		(at 122.0724 39.878 0)
@@
 		)
 	)
+	(gr_text "+"
+		(at 88.392 38.9636 180)
+		(layer "F.SilkS")
+		(effects
+			(font
+				(size 1 1)
+				(thickness 0.1)
+			)
+			(justify left bottom mirror)
+		)
+	)

Commit message: Sérigraphie complétér
Other:
- board text added: "E"
Changed lines of the file:
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@@
 		(tags "resistor")
 		(property "Reference" "R28"
-			(at -3.9624 0.0508 0)
+			(at 1.524 2.8448 90)
 			(layer "B.SilkS")
 			(effects
@@
 		)
 	)
+	(gr_text "E"
+		(at 72.4916 104.14 0)
+		(layer "B.SilkS")
+		(effects
+			(font
+				(size 1 1)
+				(thickness 0.1)
+			)
+			(justify left bottom mirror)
+		)
+	)
+	(gr_text "E"
+		(at 142.5448 81.5848 0)
+		(layer "B.SilkS")
+		(effects
+			(font
+				(size 1 1)
+				(thickness 0.1)
+			)
+			(justify left bottom mirror)
+		)
+	)
 	(gr_text "Etor"
 		(at 82.1436 112.4712 90)
@@
 		)
 	)
+	(gr_text "E"
+		(at 140.2588 81.5848 0)
+		(layer "B.SilkS")
+		(effects
+			(font
+				(size 1 1)
+				(thickness 0.1)
+			)
+			(justify left bottom mirror)
+		)
+	)
 	(gr_text "P"
 		(at 88.9508 127.1524 0)
@@
 	)
 	(gr_text "+"
+		(at 71.2724 97.9424 180)
+		(layer "B.SilkS")
+		(effects
+			(font
+				(size 1 1)
+				(thickness 0.1)
+			)
+			(justify left bottom mirror)
+		)
+	)
+	(gr_text "+"
 		(at 147.574 80.518 90)
 		(layer "B.SilkS")
@@
 		)
 	)
+	(gr_text "E"
+		(at 123.444 143.4084 0)
+		(layer "B.SilkS")
+		(effects
+			(font
+				(size 1 1)
+				(thickness 0.1)
+			)
+			(justify left bottom mirror)
+		)
+	)
 	(gr_text "Eana"
 		(at 115.2652 136.9568 90)
@@
 		)
 	)
+	(gr_text "-"
+		(at 71.3232 100.2792 180)
+		(layer "B.SilkS")
+		(effects
+			(font
+				(size 1 1)
+				(thickness 0.1)
+			)
+			(justify left bottom mirror)
+		)
+	)
 	(gr_text "K"
 		(at 122.8852 150.4188 0)
@@
 	)
 	(gr_text "+"
+		(at 71.1708 110.0328 180)
+		(layer "B.SilkS")
+		(effects
+			(font
+				(size 1 1)
+				(thickness 0.1)
+			)
+			(justify left bottom mirror)
+		)
+	)
+	(gr_text "+"
 		(at 97.8916 102.4636 90)
 		(layer "B.SilkS")
@@
 		)
 	)
+	(gr_text "E"
+		(at 72.39 116.2304 0)
+		(layer "B.SilkS")
+		(effects
+			(font
+				(size 1 1)
+				(thickness 0.1)
+			)
+			(justify left bottom mirror)
+		)
+	)
 	(gr_text "R"
 		(at 82.1944 87.5284 0)
@@
 		)
 	)
+	(gr_text "-"
+		(at 71.2216 112.3696 180)
+		(layer "B.SilkS")
+		(effects
+			(font
+				(size 1 1)
+				(thickness 0.1)
+			)
+			(justify left bottom mirror)
+		)
+	)
